File: Yamata37/yamata37.kicad_pcb (KiCad board)
At the start: 2 copper layers, 153.6 x 136.9 mm, 122 parts, among them SW1 SW_PUSH, SW10 SW_PUSH, SW11 SW_PUSH, SW13 SW_PUSH, SW14 SW_PUSH, SW15 SW_PUSH, SW16 SW_PUSH, SW17 SW_PUSH, SW18 SW_PUSH, SW19 SW_PUSH, SW20 SW_PUSH, SW21 SW_PUSH, SW22 SW_PUSH, SW23 SW_PUSH, SW24 SW_PUSH, SW25 SW_PUSH, SW26 SW_PUSH, SW27 SW_PUSH, SW28 SW_PUSH, SW29 SW_PUSH, SW3 SW_PUSH, SW30 SW_PUSH, SW31 SW_PUSH, SW32 SW_PUSH, SW33 SW_PUSH, SW34 SW_PUSH, SW35 SW_PUSH, SW36 SW_PUSH, SW37 SW_PUSH, SW38 SW_PUSH, SW4 SW_PUSH, SW5 SW_PUSH, SW6 SW_PUSH, SW8 SW_PUSH, SW9 SW_PUSH, U1 ProMicro

Commit message: rev002
Parts:
- moved LED25 0.86 mm to (71.6, 87.8)
- moved LED8 0.61 mm to (131.2, 100.1)
- moved LED15 0.54 mm to (112.2, 119.0)
- moved LED13 0.54 mm to (112.2, 80.8)
- moved LED4 0.53 mm to (150.3, 119.0)
- moved LED14 0.50 mm to (112.2, 100.1)
- moved LED35 0.32 mm to (33.3, 87.8)
- moved LED19 0.31 mm to (93.1, 100.1)
- moved LED10 0.30 mm to (131.2, 61.7)
- moved LED5 0.30 mm to (150.3, 137.9)
- moved LED20 0.26 mm to (93.1, 80.8)
- moved LED34 0.25 mm to (33.3, 68.6)
- moved LED12 0.25 mm to (112.2, 61.7)
- moved LED17 0.24 mm to (93.1, 137.9)
- moved LED21 0.24 mm to (93.1, 61.7)
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- renumbered Ref** to Ref1, Ref** to Ref2, Ref** to Ref3, Ref** to Ref4, Ref** to Ref5, Ref** to Ref6, Ref** to Ref7, Ref** to Ref8
Connections:
- U1 pad 12: unconnected-(U1-9/B5-Pad12) -> Row5
Routing:
- net GND: track 0.00 -> 1298.9 mm, vias 0 -> 52
- net VCC: track 0.00 -> 1045.9 mm, vias 0 -> 53
- net Row5: track 0.00 -> 279.9 mm, vias 0 -> 5
- net Col0: track 0.00 -> 243.8 mm, vias 0 -> 4
- net Col1: track 0.00 -> 226.0 mm, vias 0 -> 6
- net Col2: track 0.00 -> 204.9 mm, vias 0 -> 4
- net Col5: track 0.00 -> 176.3 mm, vias 0 -> 4
- net Col6: track 0.00 -> 162.5 mm, vias 0 -> 4
- net Col4: track 0.00 -> 154.0 mm, vias 0 -> 4
- net Col3: track 0.00 -> 76.8 mm, vias 0 -> 6
- net Reset: track 0.00 -> 29.1 mm, vias 0 -> 2
- net Net-(D14-A): track 0.00 -> 7.78 mm
- net Net-(D25-A): track 0.00 -> 6.98 mm
- net Net-(D2-A): track 0.00 -> 6.94 mm
- net Net-(D12-A): track 0.00 -> 6.94 mm
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
Commit message: rev002
Parts:
- turned LED1 to 180 degrees
Routing:
- net Row4: track 0.00 -> 253.6 mm, vias 0 -> 7
- net Row2: track 0.00 -> 186.5 mm, vias 0 -> 3
- net GND: track 1298.9 -> 1118.3 mm, vias 52 -> 29
- net Row1: track 0.00 -> 170.8 mm, vias 0 -> 4
- net Row3: track 0.00 -> 151.1 mm, vias 0 -> 5
- net VCC: track 1045.9 -> 916.6 mm, vias 53 -> 31
- net Row0: track 6.11 -> 120.9 mm
- net Col3: track 76.8 -> 176.8 mm
- net LED: track 0.00 -> 42.2 mm, vias 0 -> 5
- net SDA: track 0.00 -> 24.4 mm, vias 0 -> 2
- net SCL: track 0.00 -> 24.1 mm, vias 0 -> 2
- net Row5: track 279.9 -> 298.2 mm, vias 5 -> 7
