File: Yamata37/yamata37.kicad_pcb (KiCad board)
At the start: 2 copper layers, 153.6 x 136.9 mm, 122 parts, among them SW1 SW_PUSH, SW10 SW_PUSH, SW11 SW_PUSH, SW13 SW_PUSH, SW14 SW_PUSH, SW15 SW_PUSH, SW16 SW_PUSH, SW17 SW_PUSH, SW18 SW_PUSH, SW19 SW_PUSH, SW20 SW_PUSH, SW21 SW_PUSH, SW22 SW_PUSH, SW23 SW_PUSH, SW24 SW_PUSH, SW25 SW_PUSH, SW26 SW_PUSH, SW27 SW_PUSH, SW28 SW_PUSH, SW29 SW_PUSH, SW3 SW_PUSH, SW30 SW_PUSH, SW31 SW_PUSH, SW32 SW_PUSH, SW33 SW_PUSH, SW34 SW_PUSH, SW35 SW_PUSH, SW36 SW_PUSH, SW37 SW_PUSH, SW38 SW_PUSH, SW4 SW_PUSH, SW5 SW_PUSH, SW6 SW_PUSH, SW8 SW_PUSH, SW9 SW_PUSH, U1 ProMicro

Commit message: \\
Parts:
- moved LED16 0.34 mm to (111.9, 138.1), turned to 180 degrees
- moved LED15 0.27 mm to (112.0, 119.2), turned to 180 degrees
- moved LED11 0.27 mm to (112.0, 38.1), turned to 180 degrees
- moved LED12 0.27 mm to (112.0, 62.0), turned to 180 degrees
- moved LED13 0.27 mm to (112.0, 81.0), turned to 180 degrees
- moved LED14 0.27 mm to (112.0, 100.3), turned to 180 degrees
- moved LED1 0.19 mm to (150.1, 61.7), turned to 180 degrees
- moved LED2 0.18 mm to (150.1, 80.8), turned to 180 degrees
- moved LED3 0.18 mm to (150.1, 100.1), turned to 180 degrees
- moved LED4 0.18 mm to (150.1, 119.0), turned to 180 degrees
- moved LED5 0.18 mm to (150.1, 137.9), turned to 180 degrees
- turned LED23 to 180 degrees
- turned LED24 to 180 degrees
- turned LED25 to 180 degrees
- turned LED26 to 180 degrees
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Routing:
- net Row4: track 0.00 -> 255.5 mm, vias 0 -> 12
- net Row2: track 0.00 -> 200.4 mm, vias 0 -> 3
- net Row1: track 0.00 -> 168.1 mm, vias 0 -> 3
- net Row3: track 0.00 -> 150.4 mm, vias 0 -> 7
- net Row0: track 6.11 -> 129.5 mm, vias 0 -> 1
- net GND: track 1298.9 -> 1182.3 mm
- net Col3: track 76.8 -> 177.2 mm, vias 6 -> 8
- net VCC: track 1045.9 -> 1144.0 mm
- net LED: track 0.00 -> 52.2 mm, vias 0 -> 6
- net Net-(LED10-DOUT): track 0.00 -> 36.1 mm, vias 0 -> 2
- net Net-(LED32-DOUT): track 0.00 -> 32.2 mm, vias 0 -> 2
- net Net-(LED31-DOUT): track 0.00 -> 32.2 mm
- net Net-(LED29-DOUT): track 0.00 -> 32.0 mm
- net Net-(LED25-DOUT): track 0.00 -> 32.0 mm
- net Net-(LED35-DOUT): track 0.00 -> 32.0 mm
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Other:
- board size 153.6 x 136.9 mm -> 156 x 140 mm
