File: rev003/YAMATA37rev003/YAMATA37rev003.kicad_sch (KiCad schematic)
At the start: 129 parts, among them J1 TRRS_MJ-4PP-9, J2 TRRS_MJ-4PP-9, SW1 SW_PUSH, SW10 SW_PUSH, SW11 SW_DIP_x04, SW11 SW_PUSH, SW12 SW_PUSH, SW13 SW_PUSH, SW14 SW_PUSH, SW15 SW_PUSH, SW16 SW_PUSH, SW17 SW_PUSH, SW18 SW_PUSH, SW19 SW_PUSH, SW2 SW_PUSH, SW20 SW_PUSH, SW21 SW_PUSH, SW22 SW_PUSH, SW23 SW_PUSH, SW24 SW_PUSH, SW25 SW_PUSH, SW26 SW_PUSH, SW27 SW_PUSH, SW28 SW_PUSH, SW29 SW_PUSH, SW3 SW_PUSH, SW30 SW_PUSH, SW31 SW_PUSH, SW32 SW_PUSH, SW33 SW_PUSH, SW34 SW_PUSH, SW35 SW_PUSH, SW36 SW_PUSH, SW37 SW_PUSH, SW38 SW_PUSH, SW4 SW_PUSH, SW5 SW_PUSH, SW6 SW_PUSH, SW7 SW_PUSH, SW8 SW_PUSH, SW9 SW_PUSH, U1 ProMicro, U2 MCP23017_SP

Commit message: a
Parts:
- removed D28 (x2), D35, D37: D, kbd_Parts:Diode_TH_SMD, symbol Device:D
- removed LED1, LED10, LED11, LED12, LED13, LED14, LED15, LED16, LED17, LED18, LED19, LED2, LED20, LED21, LED22, LED23, LED24, LED25, LED26, LED27, LED28 (x2), LED29, LED3, LED30, LED31, LED32, LED33 (x2), LED34, LED35, LED36, LED37, LED4, LED5, LED6, LED7, LED8, LED9: LED_SK6812MINI-E, kbd_Parts:LED_SK6812MINI-E_BL_y, symbol Salicylic_kbd:LED_SK6812MINI-E
- removed SW28 (x2), SW35, SW37: SW_PUSH, kbd_SW:CherryMX_Hotswap_1u, symbol kbd:SW_PUSH
- R1, R2, R3, R4, R5: footprint kbd_Parts:Diode_TH_SMD -> Resistor_THT:R_Axial_DIN0207_L6.3mm_D2.5mm_P7.62mm_Horizontal
- SW34, SW36: footprint kbd_SW:CherryMX_Hotswap_1u -> kbd_SW:CherryMX_Hotswap_2u
- SW37: renamed from SW11; footprint Button_Switch_THT:KSA_Tactile_SPST -> Package_DIP:DIP-8_W10.16mm
Connections:
- net GND: now also R1.2, R4.2
- no-connect marks 10 -> 9
Other:
- moved on the sheet: J2, R1, R2, R3, R4, R5, SW37, U1, U2
